Commit message: update Dockerfile to install additional ROS packages and adjust xacro file mesh references to lowercase

File: meca500_description/urdf/meca500_macro.xacro (robot description, xacro)
@@ -14,5 +14,5 @@
         <origin xyz="0 0 0" rpy="0 0 0"/>
         <geometry>
-          <mesh filename="package://meca500_description/meshes/Link_0.dae"/>
+          <mesh filename="package://meca500_description/meshes/link_0.dae"/>
         </geometry>
         <material name="grey"/>
@@ -41,5 +41,5 @@
         <origin xyz="0 0 0" rpy="0 0 0"/>
         <geometry>
-          <mesh filename="package://meca500_description/meshes/Link_1.dae"/>
+          <mesh filename="package://meca500_description/meshes/link_1.dae"/>
         </geometry>
         <material name="grey"/>
@@ -62,5 +62,5 @@
         <origin xyz="0 0 0" rpy="0 0 0"/>
         <geometry>
-          <mesh filename="package://meca500_description/meshes/Link_2.dae"/>
+          <mesh filename="package://meca500_description/meshes/link_2.dae"/>
         </geometry>
         <material name="grey"/>

Commit message: feat: update Meca500 configuration and monitoring parameters for improved performance

File: meca500_description/urdf/meca500_macro.xacro (robot description, xacro)
@@ -35,5 +35,5 @@
       <child link="link_1"/>
       <origin xyz="0 0 0.135" rpy="0 0 0"/> <axis xyz="0 0 1"/>
-      <limit lower="-3.05" upper="3.05" effort="10.0" velocity="2.61"/>
+      <limit lower="-3.05" upper="3.05" effort="8.4" velocity="3.926"/>
     </joint>
     <link name="link_1">
@@ -56,5 +56,5 @@
       <child link="link_2"/>
       <origin xyz="0 0 0" rpy="0 0 0"/> <axis xyz="0 1 0"/>
-      <limit lower="-1.22" upper="1.57" effort="10.0" velocity="2.61"/>
+      <limit lower="-1.22" upper="1.57" effort="8.4" velocity="3.926"/>
     </joint>
     <link name="link_2">
@@ -83,5 +83,5 @@
       <child link="link_3"/>
       <origin xyz="0 0 0.135" rpy="0 0 0"/> <axis xyz="0 1 0"/>
-      <limit lower="-2.35" upper="1.22" effort="10.0" velocity="3.14"/>
+      <limit lower="-2.35" upper="1.22" effort="8.4" velocity="3.926"/>
     </joint>
     <link name="link_3">
@@ -110,5 +110,5 @@
       <child link="link_4"/>
       <origin xyz="0 0 0.038" rpy="0 1.5708 0"/> <axis xyz="0 0 1"/>
-      <limit lower="-2.96" upper="2.96" effort="10.0" velocity="5.23"/>
+      <limit lower="-2.96" upper="2.96" effort="1.25" velocity="6.108"/>
     </joint>
     <link name="link_4">
@@ -131,5 +131,5 @@
       <child link="link_5"/>
       <origin xyz="0 0 0.120" rpy="0 0 0"/> <axis xyz="0 1 0"/>
-      <limit lower="-2.00" upper="2.00" effort="10.0" velocity="5.23"/>
+      <limit lower="-2.00" upper="2.00" effort="1.25" velocity="6.108"/>
     </joint>
     <link name="link_5">
@@ -152,5 +152,5 @@
       <child link="link_6"/>
       <origin xyz="0 0 0.070" rpy="0 0 0"/> <axis xyz="0 0 1"/>
-      <limit lower="-6.28" upper="6.28" effort="10.0" velocity="8.72"/>
+      <limit lower="-6.28" upper="6.28" effort="0.75" velocity="8.726"/>
     </joint>
     <link name="link_6">

Commit message: feat: add inertial properties for links in Meca500 URDF macro

File: meca500_description/urdf/meca500_macro.xacro (robot description, xacro)
@@ -45,4 +45,9 @@
         <material name="grey"/>
       </visual>
+      <inertial>
+        <origin xyz="-0.00002037431904 0.002013004158 -0.02297639135" rpy="0 0 0"/>
+        <mass value="0.5431025133"/>
+        <inertia ixx="0.000915685257" ixy="5.49E-07" ixz="4.28E-07" iyy="0.0005022985235" iyz="0.00002704049297" izz="0.0008332485299"/>
+      </inertial>
       <collision>
         <origin xyz="0 0 -0.005" rpy="0 0 0"/>
@@ -66,4 +71,9 @@
         <material name="grey"/>
       </visual>
+      <inertial>
+        <origin xyz="0.04691754408 -0.005076026623 0.006334754388" rpy="0 0 0"/>
+        <mass value="1.209363494"/>
+        <inertia ixx="0.001457420783" ixy="0.00009498376543" ixz="0.00001941186918" iyy="0.003988341228" iyz="0.00001173538506" izz="0.003332374168"/>
+      </inertial>
       <collision>
         <origin xyz="-0.005 0 0.025" rpy="0 -0.23 0"/>
@@ -93,4 +103,9 @@
         <material name="grey"/>
       </visual>
+      <inertial>
+        <origin xyz="0.01508651673 0.009862786694 0.00343262302" rpy="0 0 0"/>
+        <mass value="0.8980717937"/>
+        <inertia ixx="0.0006999643903" ixy="-0.0001856385329" ixz="0.00005438767026" iyy="0.0008589980073" iyz="0.00003237561764" izz="0.00103125794"/>
+      </inertial>
       <collision>
         <origin xyz="0.017 0 0.03" rpy="0 0 0"/>
@@ -120,4 +135,9 @@
         <material name="grey"/>
       </visual>
+      <inertial>
+        <origin xyz="0.00006098710044 0.00224976832 -0.02976460875" rpy="0 0 0"/>
+        <mass value="0.2093565436"/>
+        <inertia ixx="0.0002307486811" ixy="-2.55E-07" ixz="-1.76E-07" iyy="0.0001528092348" iyz="-0.00001834894489" izz="0.0001573266858"/>
+      </inertial>
       <collision>
         <origin xyz="0 0 0.1025" rpy="0 0 0"/>
@@ -141,4 +161,9 @@
         <material name="grey"/>
       </visual>
+      <inertial>
+        <origin xyz="0.0000355330703 0.02216669127 0.003727390331" rpy="0 0 0"/>
+        <mass value="0.4881954861"/>
+        <inertia ixx="0.0004368686961" ixy="8.60E-07" ixz="-3.41E-07" iyy="0.0001588423228" iyz="0.00002942257626" izz="0.0004066877932"/>
+      </inertial>
       <collision>
         <origin xyz="0 0 0.02" rpy="0 0 0"/>
@@ -162,4 +187,9 @@
         <material name="grey"/>
       </visual>
+      <inertial>
+        <origin xyz="0 0 0" rpy="0 0 0"/>
+        <mass value="0"/>
+        <inertia ixx="0" ixy="0" ixz="0" iyy="0" iyz="0" izz="0"/>
+      </inertial>
       <collision>
         <origin xyz="0 0 -0.01" rpy="0 0 0"/>

Commit message: docs: update README.md with known issues regarding inertial parameters and control accuracy fix: correct inertial parameters in meca500_macro.xacro for improved dynamic performance

File: meca500_description/urdf/meca500_macro.xacro (robot description, xacro)
@@ -72,5 +72,5 @@
       </visual>
       <inertial>
-        <origin xyz="0.04691754408 -0.005076026623 0.006334754388" rpy="0 0 0"/>
+        <origin xyz="-0.005076026623 0.006334754388 0.04691754408" rpy="1.57 -1.57 0"/>
         <mass value="1.209363494"/>
         <inertia ixx="0.001457420783" ixy="0.00009498376543" ixz="0.00001941186918" iyy="0.003988341228" iyz="0.00001173538506" izz="0.003332374168"/>
@@ -104,5 +104,5 @@
       </visual>
       <inertial>
-        <origin xyz="0.01508651673 0.009862786694 0.00343262302" rpy="0 0 0"/>
+        <origin xyz=" 0.009862786694 0.00343262302 0.01508651673" rpy="1.57 0 0"/>
         <mass value="0.8980717937"/>
         <inertia ixx="0.0006999643903" ixy="-0.0001856385329" ixz="0.00005438767026" iyy="0.0008589980073" iyz="0.00003237561764" izz="0.00103125794"/>
@@ -136,5 +136,5 @@
       </visual>
       <inertial>
-        <origin xyz="0.00006098710044 0.00224976832 -0.02976460875" rpy="0 0 0"/>
+        <origin xyz="0.00006098710044 0.00224976832 0.08976460875" rpy="0 0 3.1415"/>
         <mass value="0.2093565436"/>
         <inertia ixx="0.0002307486811" ixy="-2.55E-07" ixz="-1.76E-07" iyy="0.0001528092348" iyz="-0.00001834894489" izz="0.0001573266858"/>
@@ -162,5 +162,5 @@
       </visual>
       <inertial>
-        <origin xyz="0.0000355330703 0.02216669127 0.003727390331" rpy="0 0 0"/>
+        <origin xyz="0.0000355330703 0.003727390331 0.02216669127" rpy="1.57 0 3.1415"/>
         <mass value="0.4881954861"/>
         <inertia ixx="0.0004368686961" ixy="8.60E-07" ixz="-3.41E-07" iyy="0.0001588423228" iyz="0.00002942257626" izz="0.0004066877932"/>

Commit message: fix: remove unnecessary whitespace in inertial origin definition

File: meca500_description/urdf/meca500_macro.xacro (robot description, xacro)
@@ -104,5 +104,5 @@
       </visual>
       <inertial>
-        <origin xyz=" 0.009862786694 0.00343262302 0.01508651673" rpy="1.57 0 0"/>
+        <origin xyz="0.009862786694 0.00343262302 0.01508651673" rpy="1.57 0 0"/>
         <mass value="0.8980717937"/>
         <inertia ixx="0.0006999643903" ixy="-0.0001856385329" ixz="0.00005438767026" iyy="0.0008589980073" iyz="0.00003237561764" izz="0.00103125794"/>
